Commit message: A4 done

File: body.urdf (robot description, URDF)
Before this commit: robot robot, 3 links, 2 joints
Links:
- added link BackLower, mass 1; collision box size=0.2 0.2 1; visual box size=0.2 0.2 1
- added link FrontLower, mass 1; collision box size=0.2 0.2 1; visual box size=0.2 0.2 1
- added link LeftLeg, mass 1; collision box size=1 0.2 0.2; visual box size=1 0.2 0.2
- added link LeftLower, mass 1; collision box size=0.2 0.2 1; visual box size=0.2 0.2 1
- added link RightLeg, mass 1; collision box size=1 0.2 0.2; visual box size=1 0.2 0.2
- added link RightLower, mass 1; collision box size=0.2 0.2 1; visual box size=0.2 0.2 1
- link BackLeg: geometry collision box size=0.2 1 0.2; visual box size=0.2 1 0.2
- link FrontLeg: geometry collision box size=0.2 1 0.2; visual box size=0.2 1 0.2
Joints:
- added joint BackLeg_BackLower: type revolute, parent BackLeg, child BackLower, origin xyz=0 -1 0 rpy=0 0 0, axis 0 1 1, limit lower=-3.14159 upper=3.14159 effort=0.0 velocity=0.0
- added joint FrontLeg_FrontLower: type revolute, parent FrontLeg, child FrontLower, origin xyz=0 1 0 rpy=0 0 0, axis 0 1 1, limit lower=-3.14159 upper=3.14159 effort=0.0 velocity=0.0
- added joint LeftLeg_LeftLower: type revolute, parent LeftLeg, child LeftLower, origin xyz=1 0 0 rpy=0 0 0, axis 0 1 1, limit lower=-3.14159 upper=3.14159 effort=0.0 velocity=0.0
- added joint RightLeg_RightLower: type revolute, parent RightLeg, child RightLower, origin xyz=-1 0 0 rpy=0 0 0, axis 0 1 1, limit lower=-3.14159 upper=3.14159 effort=0.0 velocity=0.0
- added joint Torso_LeftLeg: type revolute, parent Torso, child LeftLeg, origin xyz=0.5 0 1.0 rpy=0 0 0, axis 0 1 0, limit lower=-3.14159 upper=3.14159 effort=0.0 velocity=0.0
- added joint Torso_RightLeg: type revolute, parent Torso, child RightLeg, origin xyz=-0.5 0 1.0 rpy=0 0 0, axis 0 1 0, limit lower=-3.14159 upper=3.14159 effort=0.0 velocity=0.0
- joint Torso_BackLeg: axis 0 1 0 -> 1 0 0; origin xyz=-0.5 0 1.0 rpy=0 0 0 -> xyz=0 -0.5 1.0 rpy=0 0 0
- joint Torso_FrontLeg: axis 0 1 0 -> 1 0 0; origin xyz=0.5 0 1.0 rpy=0 0 0 -> xyz=0 0.5 1.0 rpy=0 0 0

Commit message: A5 done

File: body.urdf (robot description, URDF)
Before this commit: robot robot, 9 links, 8 joints
Links:
- removed link BackLeg
- removed link BackLower
- removed link FrontLeg
- removed link FrontLower
- removed link LeftLeg
- removed link LeftLower
- removed link RightLeg
- removed link RightLower
- added link BottomCrest, mass 1; collision box size=3 0.2 0.15; visual box size=3 0.2 0.15
- added link L1, mass 1; collision box size=0.15 0.15 0.3; visual box size=0.15 0.15 0.3
- added link L2, mass 1; collision box size=0.15 0.15 0.3; visual box size=0.15 0.15 0.3
- added link L3, mass 1; collision box size=0.15 0.15 0.3; visual box size=0.15 0.15 0.3
- added link L4, mass 1; collision box size=0.15 0.15 0.3; visual box size=0.15 0.15 0.3
- added link L5, mass 1; collision box size=0.15 0.15 0.3; visual box size=0.15 0.15 0.3
- added link L6, mass 1; collision box size=0.15 0.15 0.3; visual box size=0.15 0.15 0.3
- added link L7, mass 1; collision box size=0.15 0.15 0.3; visual box size=0.15 0.15 0.3
- added link R1, mass 1; collision box size=0.15 0.15 0.3; visual box size=0.15 0.15 0.3
- added link R2, mass 1; collision box size=0.15 0.15 0.3; visual box size=0.15 0.15 0.3
- added link R3, mass 1; collision box size=0.15 0.15 0.3; visual box size=0.15 0.15 0.3
- added link R4, mass 1; collision box size=0.15 0.15 0.3; visual box size=0.15 0.15 0.3
- added link R5, mass 1; collision box size=0.15 0.15 0.3; visual box size=0.15 0.15 0.3
- added link R6, mass 1; collision box size=0.15 0.15 0.3; visual box size=0.15 0.15 0.3
- added link R7, mass 1; collision box size=0.15 0.15 0.3; visual box size=0.15 0.15 0.3
- link Torso: geometry collision box size=3 1 0.3; visual box size=3 1 0.3
Joints:
- removed joint BackLeg_BackLower
- removed joint FrontLeg_FrontLower
- removed joint LeftLeg_LeftLower
- removed joint RightLeg_RightLower
- removed joint Torso_BackLeg
- removed joint Torso_FrontLeg
- removed joint Torso_LeftLeg
- removed joint Torso_RightLeg
- added joint Torso_BottomCrest: type revolute, parent Torso, child BottomCrest, origin xyz=0 0 0.375 rpy=0 0 0, axis 1 0 0, limit lower=-3.14159 upper=3.14159 effort=0.0 velocity=0.0
- added joint Torso_L1: type revolute, parent Torso, child L1, origin xyz=0 0.45 0.3 rpy=0 0 0, axis 0 1 0, limit lower=-3.14159 upper=3.14159 effort=0.0 velocity=0.0
- added joint Torso_L2: type revolute, parent Torso, child L2, origin xyz=0.5 0.45 0.3 rpy=0 0 0, axis 0 1 0, limit lower=-3.14159 upper=3.14159 effort=0.0 velocity=0.0
- added joint Torso_L3: type revolute, parent Torso, child L3, origin xyz=1 0.45 0.3 rpy=0 0 0, axis 0 1 0, limit lower=-3.14159 upper=3.14159 effort=0.0 velocity=0.0
- added joint Torso_L4: type revolute, parent Torso, child L4, origin xyz=1.5 0.45 0.3 rpy=0 0 0, axis 0 1 0, limit lower=-3.14159 upper=3.14159 effort=0.0 velocity=0.0
- added joint Torso_L5: type revolute, parent Torso, child L5, origin xyz=-1.5 0.45 0.3 rpy=0 0 0, axis 0 1 0, limit lower=-3.14159 upper=3.14159 effort=0.0 velocity=0.0
- added joint Torso_L6: type revolute, parent Torso, child L6, origin xyz=-1.0 0.45 0.3 rpy=0 0 0, axis 0 1 0, limit lower=-3.14159 upper=3.14159 effort=0.0 velocity=0.0
- added joint Torso_L7: type revolute, parent Torso, child L7, origin xyz=-0.5 0.45 0.3 rpy=0 0 0, axis 0 1 0, limit lower=-3.14159 upper=3.14159 effort=0.0 velocity=0.0
- added joint Torso_R1: type revolute, parent Torso, child R1, origin xyz=0 -0.45 0.3 rpy=0 0 0, axis 0 1 0, limit lower=-3.14159 upper=3.14159 effort=0.0 velocity=0.0
- added joint Torso_R2: type revolute, parent Torso, child R2, origin xyz=0.5 -0.45 0.3 rpy=0 0 0, axis 0 1 0, limit lower=-3.14159 upper=3.14159 effort=0.0 velocity=0.0
- added joint Torso_R3: type revolute, parent Torso, child R3, origin xyz=1 -0.45 0.3 rpy=0 0 0, axis 0 1 0, limit lower=-3.14159 upper=3.14159 effort=0.0 velocity=0.0
- added joint Torso_R4: type revolute, parent Torso, child R4, origin xyz=1.5 -0.45 0.3 rpy=0 0 0, axis 0 1 0, limit lower=-3.14159 upper=3.14159 effort=0.0 velocity=0.0
- added joint Torso_R5: type revolute, parent Torso, child R5, origin xyz=-1.5 -0.45 0.3 rpy=0 0 0, axis 0 1 0, limit lower=-3.14159 upper=3.14159 effort=0.0 velocity=0.0
- added joint Torso_R6: type revolute, parent Torso, child R6, origin xyz=-1.0 -0.45 0.3 rpy=0 0 0, axis 0 1 0, limit lower=-3.14159 upper=3.14159 effort=0.0 velocity=0.0
- added joint Torso_R7: type revolute, parent Torso, child R7, origin xyz=-0.5 -0.45 0.3 rpy=0 0 0, axis 0 1 0, limit lower=-3.14159 upper=3.14159 effort=0.0 velocity=0.0

Commit message: A6 complete

File: body.urdf (robot description, URDF)
Before this commit: robot robot, 16 links, 15 joints
Links:
- removed link BottomCrest
- removed link L1
- removed link L2
- removed link L3
- removed link L4
- removed link L5
- removed link L6
- removed link L7
- removed link R1
- removed link R2
- removed link R3
- removed link R4
- removed link R5
- removed link R6
- removed link R7
- removed link Torso
- added link 0, mass 1; collision box size=0.3379989599977571 0.7830167322900654 0.6002739675332478; visual box size=0.3379989599977571 0.7830167322900654 0.6002739675332478
- added link 1, mass 1; collision box size=1.1230772685105501 0.1443179825355474 1.8955975327313743; visual box size=1.1230772685105501 0.1443179825355474 1.8955975327313743
- added link 10, mass 1; collision box size=1.9991649287963997 1.2031733596492908 0.4436676350129325; visual box size=1.9991649287963997 1.2031733596492908 0.4436676350129325
- added link 11, mass 1; collision box size=1.6417603650438652 0.5764785686229321 1.321380759365528; visual box size=1.6417603650438652 0.5764785686229321 1.321380759365528
- added link 2, mass 1; collision box size=0.5881987290587916 0.23243220158829425 0.6220511457086688; visual box size=0.5881987290587916 0.23243220158829425 0.6220511457086688
- added link 3, mass 1; collision box size=1.1851717390684684 1.7796367615638709 0.19177581893456974; visual box size=1.1851717390684684 1.7796367615638709 0.19177581893456974
- added link 4, mass 1; collision box size=0.20769361328938918 0.3000437364013988 1.9584051808246865; visual box size=0.20769361328938918 0.3000437364013988 1.9584051808246865
- added link 5, mass 1; collision box size=1.2260873038662858 0.6636302484307965 1.6965568970342988; visual box size=1.2260873038662858 0.6636302484307965 1.6965568970342988
- added link 6, mass 1; collision box size=1.266918624712083 1.109028092447558 1.6377702324579477; visual box size=1.266918624712083 1.109028092447558 1.6377702324579477
- added link 7, mass 1; collision box size=1.3888252005957775 0.562628963569688 1.5329247178386836; visual box size=1.3888252005957775 0.562628963569688 1.5329247178386836
- added link 8, mass 1; collision box size=1.6065832178056787 1.779132779009054 1.5354216894238875; visual box size=1.6065832178056787 1.779132779009054 1.5354216894238875
- added link 9, mass 1; collision box size=1.666008741363715 0.05531184942437872 1.1125635815159647; visual box size=1.666008741363715 0.05531184942437872 1.1125635815159647
Joints:
- removed joint Torso_BottomCrest
- removed joint Torso_L1
- removed joint Torso_L2
- removed joint Torso_L3
- removed joint Torso_L4
- removed joint Torso_L5
- removed joint Torso_L6
- removed joint Torso_L7
- removed joint Torso_R1
- removed joint Torso_R2
- removed joint Torso_R3
- removed joint Torso_R4
- removed joint Torso_R5
- removed joint Torso_R6
- removed joint Torso_R7
- added joint 0_1: type revolute, parent 0, child 1, origin xyz=-0.9540777885116716 0 0 rpy=0 0 0, axis 0 0 1, limit lower=-3.14159 upper=3.14159 effort=0.0 velocity=0.0
- added joint 10_11: type revolute, parent 10, child 11, origin xyz=-0.6421779006456654 0 0 rpy=0 0 0, axis 0 0 1, limit lower=-3.14159 upper=3.14159 effort=0.0 velocity=0.0
- added joint 1_2: type revolute, parent 1, child 2, origin xyz=-0.0266600948035165 0 0 rpy=0 0 0, axis 0 0 1, limit lower=-3.14159 upper=3.14159 effort=0.0 velocity=0.0
- added joint 2_3: type revolute, parent 2, child 3, origin xyz=-0.8910723745390726 0 0 rpy=0 0 0, axis 0 0 1, limit lower=-3.14159 upper=3.14159 effort=0.0 velocity=0.0
- added joint 3_4: type revolute, parent 3, child 4, origin xyz=0.384892256244845 0 0 rpy=0 0 0, axis 0 0 1, limit lower=-3.14159 upper=3.14159 effort=0.0 velocity=0.0
- added joint 4_5: type revolute, parent 4, child 5, origin xyz=-1.1222404972215911 0 0 rpy=0 0 0, axis 0 0 1, limit lower=-3.14159 upper=3.14159 effort=0.0 velocity=0.0
- added joint 5_6: type revolute, parent 5, child 6, origin xyz=-0.65387497277894 0 0 rpy=0 0 0, axis 0 0 1, limit lower=-3.14159 upper=3.14159 effort=0.0 velocity=0.0
- added joint 6_7: type revolute, parent 6, child 7, origin xyz=-0.755365888239736 0 0 rpy=0 0 0, axis 0 0 1, limit lower=-3.14159 upper=3.14159 effort=0.0 velocity=0.0
- added joint 7_8: type revolute, parent 7, child 8, origin xyz=-0.9121706175077899 0 0 rpy=0 0 0, axis 0 0 1, limit lower=-3.14159 upper=3.14159 effort=0.0 velocity=0.0
- added joint 8_9: type revolute, parent 8, child 9, origin xyz=-0.8627171324608757 0 0 rpy=0 0 0, axis 0 0 1, limit lower=-3.14159 upper=3.14159 effort=0.0 velocity=0.0
- added joint 9_10: type revolute, parent 9, child 10, origin xyz=-1.1661605581145422 0 0 rpy=0 0 0, axis 0 0 1, limit lower=-3.14159 upper=3.14159 effort=0.0 velocity=0.0

Commit message: A7 done

File: body.urdf (robot description, URDF)
Before this commit: robot robot, 12 links, 11 joints
Links:
- added link 12, mass 1; collision box size=1.9451231048660877 1.0652436899206743 0.3181756424809503; visual box size=1.9451231048660877 1.0652436899206743 0.3181756424809503
- added link 13, mass 1; collision box size=0.6083026570050492 1.2173767055419917 0.0766292445088228; visual box size=0.6083026570050492 1.2173767055419917 0.0766292445088228
- added link 14, mass 1; collision box size=1.9572815758450268 0.6926948935181043 0.5135646789101984; visual box size=1.9572815758450268 0.6926948935181043 0.5135646789101984
- link 0: geometry collision box size=1.063952072594976 0.25872262749530495 1.6838047168389798; visual box size=1.063952072594976 0.25872262749530495 1.6838047168389798
- link 1: geometry collision box size=0.06754519937325631 1.1175553036758352 0.9393517230728632; visual box size=0.06754519937325631 1.1175553036758352 0.9393517230728632
- link 10: geometry collision box size=1.0073974940589954 1.2095391306688328 0.6620203332646275; visual box size=1.0073974940589954 1.2095391306688328 0.6620203332646275
- link 11: geometry collision box size=0.09220134820631354 0.23697006382837515 0.3558849625600842; visual box size=0.09220134820631354 0.23697006382837515 0.3558849625600842
- link 2: geometry collision box size=1.3027385914932283 0.1889099209121603 0.08482354334125719; visual box size=1.3027385914932283 0.1889099209121603 0.08482354334125719
- link 3: geometry collision box size=1.2365606737470731 1.4672482716559705 1.4156915848169989; visual box size=1.2365606737470731 1.4672482716559705 1.4156915848169989
- link 4: geometry collision box size=1.51072738355852 1.4984206327195662 1.9262153559135777; visual box size=1.51072738355852 1.4984206327195662 1.9262153559135777
- link 5: geometry collision box size=1.74523135532142 0.6568052861750389 0.9390704885444321; visual box size=1.74523135532142 0.6568052861750389 0.9390704885444321
- link 6: geometry collision box size=1.798706785605958 1.1236934292089735 1.2078490206758385; visual box size=1.798706785605958 1.1236934292089735 1.2078490206758385
- link 7: geometry collision box size=1.0154486865459718 0.773470757239284 0.8656978064728835; visual box size=1.0154486865459718 0.773470757239284 0.8656978064728835
- link 8: geometry collision box size=1.7230033736860038 0.3027571768502122 1.7472052230559263; visual box size=1.7230033736860038 0.3027571768502122 1.7472052230559263
- link 9: geometry collision box size=0.9550913432732264 0.39733565738084686 1.8907877140164164; visual box size=0.9550913432732264 0.39733565738084686 1.8907877140164164
Joints:
- removed joint 10_11
- removed joint 2_3
- removed joint 4_5
- removed joint 5_6
- removed joint 6_7
- removed joint 7_8
- removed joint 9_10
- added joint 0_6: type revolute, parent 0, child 6, origin xyz=0.16459867979199705 0 0 rpy=0 0 0, axis 0 1 1, limit lower=-3.14159 upper=3.14159 effort=0.0 velocity=0.0
- added joint 0_8: type revolute, parent 0, child 8, origin xyz=-0.20245038575197416 0 0 rpy=0 0 0, axis 0 1 1, limit lower=-3.14159 upper=3.14159 effort=0.0 velocity=0.0
- added joint 1_3: type revolute, parent 1, child 3, origin xyz=-0.5507351375002802 0 0 rpy=0 0 0, axis 0 1 1, limit lower=-3.14159 upper=3.14159 effort=0.0 velocity=0.0
- added joint 3_11: type revolute, parent 3, child 11, origin xyz=1.1904599996439162 0 0 rpy=0 0 0, axis 0 1 1, limit lower=-3.14159 upper=3.14159 effort=0.0 velocity=0.0
- added joint 3_5: type revolute, parent 3, child 5, origin xyz=0 -1.138845628568451 0 rpy=0 0 0, axis 1 0 1, limit lower=-3.14159 upper=3.14159 effort=0.0 velocity=0.0
- added joint 4_14: type revolute, parent 4, child 14, origin xyz=0 1.152073185960514 0 rpy=0 0 0, axis 1 0 1, limit lower=-3.14159 upper=3.14159 effort=0.0 velocity=0.0
- added joint 5_7: type revolute, parent 5, child 7, origin xyz=0 -0.27006990755539684 0 rpy=0 0 0, axis 1 0 1, limit lower=-3.14159 upper=3.14159 effort=0.0 velocity=0.0
- added joint 6_12: type revolute, parent 6, child 12, origin xyz=0 -0.5910715842486364 0 rpy=0 0 0, axis 1 0 1, limit lower=-3.14159 upper=3.14159 effort=0.0 velocity=0.0
- added joint 7_10: type revolute, parent 7, child 10, origin xyz=0 0 -0.5346876398405698 rpy=0 0 0, axis 1 1 0, limit lower=-3.14159 upper=3.14159 effort=0.0 velocity=0.0
- added joint 7_13: type revolute, parent 7, child 13, origin xyz=0 -0.16478240446828818 0 rpy=0 0 0, axis 1 0 1, limit lower=-3.14159 upper=3.14159 effort=0.0 velocity=0.0
- joint 0_1: axis 0 0 1 -> 1 0 1; origin xyz=-0.9540777885116716 0 0 rpy=0 0 0 -> xyz=0 0.30005502434261266 0 rpy=0 0 0
- joint 1_2: axis 0 0 1 -> 1 1 0; origin xyz=-0.0266600948035165 0 0 rpy=0 0 0 -> xyz=0 0 -0.8969399514022346 rpy=0 0 0
- joint 3_4: axis 0 0 1 -> 1 0 1; origin xyz=0.384892256244845 0 0 rpy=0 0 0 -> xyz=0 0.7180379552961874 0 rpy=0 0 0
- joint 8_9: axis 0 0 1 -> 1 1 0; origin xyz=-0.8627171324608757 0 0 rpy=0 0 0 -> xyz=0 0 -0.8018113660477181 rpy=0 0 0

Commit message: adjustment of bot constructions

File: body.urdf (robot description, URDF)
Before this commit: robot robot, 15 links, 14 joints
Links:
- removed link 10
- removed link 11
- removed link 12
- removed link 13
- removed link 14
- removed link 9
- link 0: geometry collision box size=0.4351169129161945 0.6601078441244896 0.9889013940169795; visual box size=0.4351169129161945 0.6601078441244896 0.9889013940169795
- link 1: geometry collision box size=0.9271298411047788 0.9336431893243511 0.5110548198932057; visual box size=0.9271298411047788 0.9336431893243511 0.5110548198932057
- link 2: geometry collision box size=0.48381573315469917 0.9933144452956888 0.770130733688341; visual box size=0.48381573315469917 0.9933144452956888 0.770130733688341
- link 3: geometry collision box size=0.91364721610531 0.21309508882706246 0.3718937878130195; visual box size=0.91364721610531 0.21309508882706246 0.3718937878130195
- link 4: geometry collision box size=0.9776583541234518 0.6853691677864258 0.332503201073314; visual box size=0.9776583541234518 0.6853691677864258 0.332503201073314
- link 5: geometry collision box size=0.9155431524544131 0.935355813379583 0.6347562652237182; visual box size=0.9155431524544131 0.935355813379583 0.6347562652237182
- link 6: geometry collision box size=0.9540925676238194 0.9484342896033433 0.7628426317755883; visual box size=0.9540925676238194 0.9484342896033433 0.7628426317755883
- link 7: geometry collision box size=0.7197060487089006 0.5151642302839576 0.29009051621196486; visual box size=0.7197060487089006 0.5151642302839576 0.29009051621196486
- link 8: geometry collision box size=0.35349565855283793 0.2997570764439906 0.8925552327746302; visual box size=0.35349565855283793 0.2997570764439906 0.8925552327746302
Joints:
- removed joint 0_8
- removed joint 1_3
- removed joint 3_11
- removed joint 3_4
- removed joint 3_5
- removed joint 4_14
- removed joint 5_7
- removed joint 6_12
- removed joint 7_10
- removed joint 7_13
- removed joint 8_9
- added joint 0_7: type revolute, parent 0, child 7, origin xyz=0 -0.072471806920266 0 rpy=0 0 0, axis 1 0 1, limit lower=-3.14159 upper=3.14159 effort=0.0 velocity=0.0
- added joint 2_3: type revolute, parent 2, child 3, origin xyz=0 0.3901096782343132 0 rpy=0 0 0, axis 1 0 1, limit lower=-3.14159 upper=3.14159 effort=0.0 velocity=0.0
- added joint 2_4: type revolute, parent 2, child 4, origin xyz=0 0 0.07565626604069259 rpy=0 0 0, axis 1 1 0, limit lower=-3.14159 upper=3.14159 effort=0.0 velocity=0.0
- added joint 2_5: type revolute, parent 2, child 5, origin xyz=-0.21586370964985696 0 0 rpy=0 0 0, axis 0 1 1, limit lower=-3.14159 upper=3.14159 effort=0.0 velocity=0.0
- added joint 4_8: type revolute, parent 4, child 8, origin xyz=0 0 0.04255156067441079 rpy=0 0 0, axis 1 1 0, limit lower=-3.14159 upper=3.14159 effort=0.0 velocity=0.0
- joint 0_1: axis 1 0 1 -> 0 1 1; origin xyz=0 0.30005502434261266 0 rpy=0 0 0 -> xyz=-0.24600646409429217 0 0 rpy=0 0 0
- joint 0_6: origin xyz=0.16459867979199705 0 0 rpy=0 0 0 -> xyz=0.2594878273538125 0 0 rpy=0 0 0
- joint 1_2: axis 1 1 0 -> 1 0 1; origin xyz=0 0 -0.8969399514022346 rpy=0 0 0 -> xyz=0 -0.029835627985668856 0 rpy=0 0 0

Commit message: rel positions added

File: body.urdf (robot description, URDF)
Before this commit: robot robot, 9 links, 8 joints
Links:
- link 0: geometry collision box size=0.2770893645054697 0.5267019104447999 0.45580660931340083; visual box size=0.2770893645054697 0.5267019104447999 0.45580660931340083
- link 1: geometry collision box size=0.9865271400168634 0.5663405116724005 0.6816421315606345; visual box size=0.9865271400168634 0.5663405116724005 0.6816421315606345
- link 2: geometry collision box size=0.7607922959931035 0.44113392738188156 0.2449949608388482; visual box size=0.7607922959931035 0.44113392738188156 0.2449949608388482
- link 3: geometry collision box size=0.6747080048086389 0.7420916362401246 0.24400025052312416; visual box size=0.6747080048086389 0.7420916362401246 0.24400025052312416
- link 4: geometry collision box size=0.3230439313614805 0.8600121226892747 0.6136502174984142; visual box size=0.3230439313614805 0.8600121226892747 0.6136502174984142
- link 5: geometry collision box size=0.5357286430179045 0.2629998775769384 0.344599164137778; visual box size=0.5357286430179045 0.2629998775769384 0.344599164137778
- link 6: geometry collision box size=0.6209885790029843 0.458653308540276 0.43112812756215474; visual box size=0.6209885790029843 0.458653308540276 0.43112812756215474
- link 7: geometry collision box size=0.981312448525876 0.9296972086885622 0.949884837281495; visual box size=0.981312448525876 0.9296972086885622 0.949884837281495
- link 8: geometry collision box size=0.789923609032259 0.48093640834863804 0.3646217531831103; visual box size=0.789923609032259 0.48093640834863804 0.3646217531831103
Joints:
- removed joint 0_6
- removed joint 0_7
- removed joint 2_3
- removed joint 2_5
- removed joint 4_8
- added joint 0_3: type revolute, parent 0, child 3, origin xyz=0 -0.3710458181200623 0.12200012526156208 rpy=0 0 0, axis 1 0 1, limit lower=-3.14159 upper=3.14159 effort=0.0 velocity=0.0
- added joint 2_6: type revolute, parent 2, child 6, origin xyz=-0.7607922959931035 0 0 rpy=0 0 0, axis 0 1 1, limit lower=-3.14159 upper=3.14159 effort=0.0 velocity=0.0
- added joint 3_8: type revolute, parent 3, child 8, origin xyz=0.33735400240431945 -0.3710458181200623 0 rpy=0 0 0, axis 0 1 1, limit lower=-3.14159 upper=3.14159 effort=0.0 velocity=0.0
- added joint 4_5: type revolute, parent 4, child 5, origin xyz=-0.3230439313614805 -0.43000606134463737 0 rpy=0 0 0, axis 0 1 1, limit lower=-3.14159 upper=3.14159 effort=0.0 velocity=0.0
- added joint 6_7: type revolute, parent 6, child 7, origin xyz=-0.31049428950149216 0 0.21556406378107737 rpy=0 0 0, axis 1 1 0, limit lower=-3.14159 upper=3.14159 effort=0.0 velocity=0.0
- joint 0_1: axis 0 1 1 -> 1 1 0; origin xyz=-0.24600646409429217 0 0 rpy=0 0 0 -> xyz=0 0 0.6816421315606345 rpy=0 0 0
- joint 1_2: axis 1 0 1 -> 0 1 1; origin xyz=0 -0.029835627985668856 0 rpy=0 0 0 -> xyz=-0.4932635700084317 0 0.34082106578031723 rpy=0 0 0
- joint 2_4: axis 1 1 0 -> 1 0 1; origin xyz=0 0 0.07565626604069259 rpy=0 0 0 -> xyz=-0.38039614799655175 -0.22056696369094078 0 rpy=0 0 0
