Commit message: return to parallelism

File: body.urdf (robot description, URDF)
Before this commit: robot robot, 9 links, 8 joints
Links:
- added link 10, mass 1; collision box size=0.9694392508785372 0.7290080036357873 0.9641799724520921; visual box size=0.9694392508785372 0.7290080036357873 0.9641799724520921
- added link 11, mass 1; collision box size=0.7469996386251059 0.8543474139729672 0.961162246191682; visual box size=0.7469996386251059 0.8543474139729672 0.961162246191682
- added link 9, mass 1; collision box size=0.8381993494092528 0.33824723423262226 0.9236075262027226; visual box size=0.8381993494092528 0.33824723423262226 0.9236075262027226
- link 0: geometry collision box size=0.9897313380985655 0.8903261293607281 0.45901119441740645; visual box size=0.9897313380985655 0.8903261293607281 0.45901119441740645
- link 1: geometry collision box size=0.7966883839514765 0.7248304741125293 0.25519082352664785; visual box size=0.7966883839514765 0.7248304741125293 0.25519082352664785
- link 2: geometry collision box size=0.4298344913420775 0.651202982428998 0.34471491364128837; visual box size=0.4298344913420775 0.651202982428998 0.34471491364128837
- link 3: geometry collision box size=0.28712112163746095 0.43351684903311893 0.27600640240445484; visual box size=0.28712112163746095 0.43351684903311893 0.27600640240445484
- link 4: geometry collision box size=0.28186571716642544 0.3219256324516315 0.7534101182116573; visual box size=0.28186571716642544 0.3219256324516315 0.7534101182116573
- link 5: geometry collision box size=0.5997555214866283 0.5022451519606439 0.6926973542033974; visual box size=0.5997555214866283 0.5022451519606439 0.6926973542033974
- link 6: geometry collision box size=0.7516729418014507 0.8723696433782446 0.8031147996445778; visual box size=0.7516729418014507 0.8723696433782446 0.8031147996445778
- link 7: geometry collision box size=0.7888043663998758 0.6690156650462621 0.6967228151801473; visual box size=0.7888043663998758 0.6690156650462621 0.6967228151801473
- link 8: geometry collision box size=0.6267398277371363 0.34877679895115166 0.874309014264903; visual box size=0.6267398277371363 0.34877679895115166 0.874309014264903
Joints:
- removed joint 1_2
- removed joint 2_4
- removed joint 2_6
- removed joint 3_8
- removed joint 4_5
- removed joint 6_7
- added joint 0_2: type revolute, parent 0, child 2, origin xyz=0 0.325601491214499 2.1723574568206443 rpy=0 0 0, axis 1 0 1, limit lower=-3.14159 upper=3.14159 effort=0.0 velocity=0.0
- added joint 0_8: type revolute, parent 0, child 8, origin xyz=-0.31336991386856816 0 2.4371545071324516 rpy=0 0 0, axis 0 1 1, limit lower=-3.14159 upper=3.14159 effort=0.0 velocity=0.0
- added joint 0_9: type revolute, parent 0, child 9, origin xyz=0.4190996747046264 0 2.4618037631013614 rpy=0 0 0, axis 0 1 1, limit lower=-3.14159 upper=3.14159 effort=0.0 velocity=0.0
- added joint 1_4: type revolute, parent 1, child 4, origin xyz=0 0.36241523705626466 -0.12759541176332392 rpy=0 0 0, axis 1 0 1, limit lower=-3.14159 upper=3.14159 effort=0.0 velocity=0.0
- added joint 1_6: type revolute, parent 1, child 6, origin xyz=0 0 -0.25519082352664785 rpy=0 0 0, axis 1 1 0, limit lower=-3.14159 upper=3.14159 effort=0.0 velocity=0.0
- added joint 3_5: type revolute, parent 3, child 5, origin xyz=0.14356056081873048 -0.21675842451655947 0 rpy=0 0 0, axis 0 1 1, limit lower=-3.14159 upper=3.14159 effort=0.0 velocity=0.0
- added joint 3_7: type revolute, parent 3, child 7, origin xyz=0 -0.21675842451655947 0.13800320120222742 rpy=0 0 0, axis 1 1 0, limit lower=-3.14159 upper=3.14159 effort=0.0 velocity=0.0
- added joint 4_11: type revolute, parent 4, child 11, origin xyz=-0.14093285858321272 0.16096281622581576 0 rpy=0 0 0, axis 0 1 1, limit lower=-3.14159 upper=3.14159 effort=0.0 velocity=0.0
- added joint 6_10: type revolute, parent 6, child 10, origin xyz=-0.37583647090072536 0 -0.4015573998222889 rpy=0 0 0, axis 0 1 1, limit lower=-3.14159 upper=3.14159 effort=0.0 velocity=0.0
- joint 0_1: origin xyz=0 0 0.6816421315606345 rpy=0 0 0 -> xyz=0 0 2 rpy=0 0 0
- joint 0_3: origin xyz=0 -0.3710458181200623 0.12200012526156208 rpy=0 0 0 -> xyz=0 -0.21675842451655947 2.1380032012022276 rpy=0 0 0
