Commit message: insane robots activated
they fucking cartwheel what

File: artificialLifeFinalProjectStuff/AReallyGoodRobot/body940.urdf (robot description, URDF)
Before this commit: robot robot, 12 links, 11 joints
Links:
- link 0: geometry collision box size=0.5011821767277225 0.5285243140091682 0.41477200967601036; visual box size=0.5011821767277225 0.5285243140091682 0.41477200967601036
- link 1: geometry collision box size=0.27757166527625626 0.7133329162206619 0.8006634838140008; visual box size=0.27757166527625626 0.7133329162206619 0.8006634838140008
- link 10: geometry collision box size=0.27161792339240975 0.693474259087962 0.40903856132479777; visual box size=0.27161792339240975 0.693474259087962 0.40903856132479777
- link 11: geometry collision box size=0.7897430338513991 0.9712281098480366 0.502222726612255; visual box size=0.7897430338513991 0.9712281098480366 0.502222726612255
- link 2: geometry collision box size=0.5363184134969228 0.9339134359902164 0.2064780461482644; visual box size=0.5363184134969228 0.9339134359902164 0.2064780461482644
- link 3: geometry collision box size=0.9649784364290439 0.6613505639834769 0.20124806525672512; visual box size=0.9649784364290439 0.6613505639834769 0.20124806525672512
- link 4: geometry collision box size=0.3176150633463003 0.5892648527397055 0.3913099921310197; visual box size=0.3176150633463003 0.5892648527397055 0.3913099921310197
- link 5: geometry collision box size=0.4521658178081361 0.42035688909091445 0.8294911220196879; visual box size=0.4521658178081361 0.42035688909091445 0.8294911220196879
- link 6: geometry collision box size=0.7433575190801383 0.3225271553034874 0.7449966678807638; visual box size=0.7433575190801383 0.3225271553034874 0.7449966678807638
- link 7: geometry collision box size=0.6612627076354377 0.37825247660283523 0.9845276965075074; visual box size=0.6612627076354377 0.37825247660283523 0.9845276965075074
- link 8: geometry collision box size=0.3556557359018065 0.9830085102110955 0.32730247908580035; visual box size=0.3556557359018065 0.9830085102110955 0.32730247908580035
- link 9: geometry collision box size=0.5560123814859855 0.5637297365974714 0.9380001346151976; visual box size=0.5560123814859855 0.5637297365974714 0.9380001346151976
Joints:
- removed joint 0_8
- removed joint 0_9
- removed joint 1_4
- removed joint 1_6
- removed joint 4_11
- removed joint 6_10
- added joint 2_4: type revolute, parent 2, child 4, origin xyz=0 0.4669567179951082 0.1032390230741322 rpy=0 0 0, axis 1 1 0, limit lower=-3.14159 upper=3.14159 effort=0.0 velocity=0.0
- added joint 2_6: type revolute, parent 2, child 6, origin xyz=0 0.4669567179951082 -0.1032390230741322 rpy=0 0 0, axis 1 1 0, limit lower=-3.14159 upper=3.14159 effort=0.0 velocity=0.0
- added joint 2_8: type revolute, parent 2, child 8, origin xyz=-0.2681592067484614 0.4669567179951082 0 rpy=0 0 0, axis 0 1 1, limit lower=-3.14159 upper=3.14159 effort=0.0 velocity=0.0
- added joint 6_9: type revolute, parent 6, child 9, origin xyz=0 -0.1612635776517437 -0.3724983339403819 rpy=0 0 0, axis 1 0 1, limit lower=-3.14159 upper=3.14159 effort=0.0 velocity=0.0
- added joint 9_10: type revolute, parent 9, child 10, origin xyz=-0.5560123814859855 -0.2818648682987357 0 rpy=0 0 0, axis 0 1 1, limit lower=-3.14159 upper=3.14159 effort=0.0 velocity=0.0
- added joint 9_11: type revolute, parent 9, child 11, origin xyz=0 -0.2818648682987357 -0.4690000673075988 rpy=0 0 0, axis 1 1 0, limit lower=-3.14159 upper=3.14159 effort=0.0 velocity=0.0
- joint 0_1: axis 1 1 0 -> 0 1 1; origin xyz=0 0 2 rpy=0 0 0 -> xyz=0.13878583263812813 0 2.4003317419070003 rpy=0 0 0
- joint 0_2: origin xyz=0 0.325601491214499 2.1723574568206443 rpy=0 0 0 -> xyz=0 0.4669567179951082 2.1032390230741322 rpy=0 0 0
- joint 0_3: axis 1 0 1 -> 1 1 0; origin xyz=0 -0.21675842451655947 2.1380032012022276 rpy=0 0 0 -> xyz=0 0 2 rpy=0 0 0
- joint 3_5: axis 0 1 1 -> 1 0 1; origin xyz=0.14356056081873048 -0.21675842451655947 0 rpy=0 0 0 -> xyz=0 -0.33067528199173846 -0.10062403262836256 rpy=0 0 0
- joint 3_7: axis 1 1 0 -> 0 1 1; origin xyz=0 -0.21675842451655947 0.13800320120222742 rpy=0 0 0 -> xyz=-0.48248921821452195 0 -0.10062403262836256 rpy=0 0 0
